File: EAA690_RFID_In.sch (EAGLE design)
At the start: 3 parts, among them T1 TIP31

Commit message: Minor changes
Parts:
- added BAT1: (no value), special:BATTERY
- added D1: (no value), diode:ZENER-DIODESOD64-12
- added S1: (no value), SparkFun-Electromechanical:SWITCH-SPDTPTH
Connections:
- new net N$11: D1.A, D1.C, S1.S, T1.E
- new net N$12: BAT1.-
- new net N$15: BAT1.+, S1.P, T1.C
Other:
- moved on the sheet: T1
Changed lines of the file:
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@@
 <part name="X1" library="SparkFun-Connectors" deviceset="DB9" device="FEMALE"/>
 <part name="T1" library="transistor" deviceset="TIP31" device=""/>
+<part name="BAT1" library="special" deviceset="BATTERY" device=""/>
+<part name="S1" library="SparkFun-Electromechanical" deviceset="SWITCH-SPDT" device="PTH"/>
+<part name="D1" library="diode" deviceset="ZENER-DIODE" device="SOD64-12"/>
 </parts>
 <sheets>
@@
 <instance part="U$1" gate="G$1" x="15.24" y="68.58"/>
 <instance part="X1" gate="G$1" x="66.04" y="66.04"/>
-<instance part="T1" gate="G$1" x="43.18" y="27.94"/>
+<instance part="T1" gate="G$1" x="43.18" y="35.56"/>
+<instance part="BAT1" gate="G$1" x="60.96" y="45.72"/>
+<instance part="S1" gate="1" x="53.34" y="35.56"/>
+<instance part="D1" gate="G$1" x="50.8" y="27.94"/>
 </instances>
 <busses>
@@
 <pinref part="U$1" gate="G$1" pin="D2"/>
 <wire x1="27.94" y1="78.74" x2="40.64" y2="78.74" width="0.1524" layer="91"/>
-<wire x1="40.64" y1="78.74" x2="40.64" y2="27.94" width="0.1524" layer="91"/>
+<wire x1="40.64" y1="78.74" x2="40.64" y2="35.56" width="0.1524" layer="91"/>
 <pinref part="T1" gate="G$1" pin="B"/>
 </segment>
@@
 </segment>
 </net>
+<net name="N$12" class="0">
+<segment>
+<pinref part="BAT1" gate="G$1" pin="-"/>
+<wire x1="66.04" y1="45.72" x2="66.04" y2="20.32" width="0.1524" layer="91"/>
+</segment>
+</net>
+<net name="N$15" class="0">
+<segment>
+<pinref part="T1" gate="G$1" pin="C"/>
+<wire x1="50.8" y1="45.72" x2="45.72" y2="45.72" width="0.1524" layer="91"/>
+<pinref part="S1" gate="1" pin="P"/>
+<wire x1="50.8" y1="35.56" x2="50.8" y2="45.72" width="0.1524" layer="91"/>
+<junction x="50.8" y="45.72"/>
+<wire x1="45.72" y1="40.64" x2="45.72" y2="45.72" width="0.1524" layer="91"/>
+<pinref part="BAT1" gate="G$1" pin="+"/>
+<wire x1="50.8" y1="45.72" x2="55.88" y2="45.72" width="0.1524" layer="91"/>
+</segment>
+</net>
+<net name="N$11" class="0">
+<segment>
+<pinref part="S1" gate="1" pin="S"/>
+<wire x1="58.42" y1="33.02" x2="58.42" y2="27.94" width="0.1524" layer="91"/>
+<pinref part="T1" gate="G$1" pin="E"/>
+<wire x1="45.72" y1="30.48" x2="45.72" y2="27.94" width="0.1524" layer="91"/>
+<pinref part="D1" gate="G$1" pin="A"/>
+<wire x1="45.72" y1="27.94" x2="48.26" y2="27.94" width="0.1524" layer="91"/>
+<pinref part="D1" gate="G$1" pin="C"/>
+<wire x1="48.26" y1="27.94" x2="53.34" y2="27.94" width="0.1524" layer="91"/>
+<wire x1="53.34" y1="27.94" x2="58.42" y2="27.94" width="0.1524" layer="91"/>
+<wire x1="58.42" y1="27.94" x2="58.42" y2="20.32" width="0.1524" layer="91"/>
+<junction x="58.42" y="27.94"/>
+</segment>
+</net>
